File: PCB/keobard.kicad_pcb (KiCad board)
At the start: 2 copper layers, 353.3 x 102.1 mm, 134 parts, among them J2 Conn_01x04_MountingPin, SW2 RotaryEncoder_Switch

Commit message: e
Parts:
- D58: moved to B.Cu
- J2, SW2: moved to F.Cu
- moved SW2 15.0 mm to (319.5, 62.8), turned to 0 degrees
- moved J2 8.80 mm to (325.2, 84.5)
Routing:
- net COL13: track 508.7 -> 440.8 mm, vias 4 -> 6
- net GND: track 181.6 -> 144.8 mm
- net ENCA: track 38.8 -> 22.3 mm
- net COL15: track 89.3 -> 75.5 mm
- net ENCB: track 31.5 -> 22.1 mm
- net SDA: track 26.1 -> 31.0 mm, vias 2 -> 0
- net Net-(D58-A): track 27.6 -> 25.8 mm, vias 2 -> 1
- net VCC: track 36.9 -> 35.2 mm
- net SLC: track 25.3 -> 26.3 mm
